File: boards/field_device/field_device.kicad_pcb (KiCad board)
At the start: 4 copper layers, 50 x 60 mm, 56 parts, among them SW1 TS-1088-AR02016, U1 CHT20MEMS, U2 STM32C051F8P6, U3 SPA06-003, U4 CN3163, U6 SX1262IMLTRT, U7 TPS63900, Y1 X322532MMB4SI

Commit message: update
Parts:
- moved J2 14.5 mm to (34.5, 15.0)
- moved C10 12.0 mm to (18.4, 32.9)
- moved C8 12.0 mm to (18.7, 20.0)
- moved D2 12.0 mm to (16.2, 25.1)
- moved R15 12.0 mm to (16.8, 27.6)
- moved R18 12.0 mm to (19.2, 29.1)
- moved U7 12.0 mm to (20.8, 32.8)
- moved C7 12.0 mm to (22.8, 20.0)
- moved D3 12.0 mm to (16.2, 21.5)
- moved L1 12.0 mm to (20.9, 36.9)
- moved R14 12.0 mm to (25.1, 23.4)
- moved R16 12.0 mm to (22.6, 29.1)
- moved U4 12.0 mm to (20.8, 23.4)
- moved C9 12.0 mm to (23.3, 32.9)
- moved BT1 11.9 mm to (16.6, 14.7)
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Routing:
- net /MCU/LOG_MCU_TX_DEBUGGER_RX: track 55.4 -> 35.0 mm, vias 1 -> 2
- net /MCU/LOG_MCU_RX_DEBUGGER_TX: track 48.8 -> 40.0 mm, vias 2 -> 1
- net /MCU/NRST: track 34.2 -> 41.6 mm
- net /MCU/SCL_bus: track 27.3 -> 32.8 mm
- net /MCU/SDA_bus: track 26.4 -> 31.8 mm
- net GND: track 73.3 -> 69.2 mm, vias 23 -> 24
- net /MCU/MCU_MISO: track 30.9 -> 29.0 mm
- net +3.3V: track 41.2 -> 39.6 mm
- net /power_source/solar_pwr: track 21.2 -> 19.9 mm
- net /power_source/regulator/Vin: track 35.3 -> 34.4 mm
- net /MCU/LOG_MCU_RX: track 7.17 -> 7.77 mm
Other:
- board text removed: "All the words I left unsaid that day"
- board text removed: "Didn't you see the news today?"
- board text removed: "I heard they said it looked like rain"
- board text removed: "Stained the sidewalk drop-by-drop"
- board text removed: "with gray."
